Commit message: restructuring but everything broke

File: mobile_base_description/urdf/gazebo/control.xacro (robot description, xacro)
@@ -2,9 +2,9 @@
 <!-- This file contains the Gazebo controller interface. -->
 <robot name="mobile_base" xmlns:xacro="http://www.ros.org/wiki/xacro">
-   <xacro:macro name="load_gazebo_ros_control">
+   <xacro:macro name="load_gazebo_ros_control" params="ns:=mobile_base">
     <gazebo>
       <plugin name="gazebo_ros_control" filename="libgazebo_ros_control.so">
         <robotNamespace>/mobile_base</robotNamespace>
-        <controlPeriod>0.001</controlPeriod>
+        <!-- <controlPeriod>0.001</controlPeriod> -->
         <robotParam>robot_description</robotParam>
         <robotSimType>gazebo_ros_control/DefaultRobotHWSim</robotSimType>

File: mobile_base_description/urdf/mobile_base.urdf.xacro (robot description, xacro)
@@ -50,4 +50,5 @@
                 <material name="green"/>
             </visual>
+            <inertial/>
         </link>
         <gazebo reference="base">

File: mobile_base_description/urdf/mobile_base_standalone.urdf.xacro (robot description, xacro)
@@ -1,9 +1,13 @@
 <?xml version="1.0"?>
 <robot xmlns:xacro="http://www.ros.org/wiki/xacro" name="mobile_base">
-	<!-- Includes -->
-  <xacro:include filename="$(find mobile_base_description)/urdf/properties.urdf.xacro" />
-  <xacro:include filename="$(find mobile_base_description)/urdf/mobile_base.urdf.xacro"/>
-  <!-- Arguments -->
-  <xacro:arg name="wheel_joint_type"  default="fixed"/> <!-- continuous for gazebo -->
-  <xacro:mobile_base wheel_joint_type="$(arg wheel_joint_type)"/>
+  <!-- Includes -->
+  <xacro:arg name="simulation" 			default="false"/>
+  <xacro:arg name="wheel_joint_type"  	default="fixed"/> <!-- continuous for gazebo -->
+  <!-- Load the base -->
+  <xacro:include filename="$(find mobile_base_description)/urdf/mobile_base_macro.urdf.xacro"/>
+  <xacro:load_mobile_base simulation="$(arg simulation)" wheel_joint_type="$(arg wheel_joint_type)"/>
+  <!-- Ros control -->
+  <xacro:if value="$(arg simulation)">
+    <xacro:include filename="$(find mobile_base_description)/urdf/gazebo/control.xacro"/>
+  </xacro:if>
 </robot>

Commit message: working restructuring and skid steer

File: mobile_base_description/urdf/gazebo/control.xacro (robot description, xacro)
@@ -1,11 +1,9 @@
 <?xml version="1.0"?>
 <!-- This file contains the Gazebo controller interface. -->
-<robot name="mobile_base" xmlns:xacro="http://www.ros.org/wiki/xacro">
-   <xacro:macro name="load_gazebo_ros_control" params="ns:=mobile_base">
+<robot xmlns:xacro="http://www.ros.org/wiki/xacro">
+   <xacro:macro name="load_gazebo_ros_control" params="ns:='' ">
     <gazebo>
       <plugin name="gazebo_ros_control" filename="libgazebo_ros_control.so">
-        <robotNamespace>/mobile_base</robotNamespace>
-        <!-- <controlPeriod>0.001</controlPeriod> -->
-        <robotParam>robot_description</robotParam>
+        <robotNamespace>${ns}</robotNamespace>
         <robotSimType>gazebo_ros_control/DefaultRobotHWSim</robotSimType>
       </plugin>

File: mobile_base_description/urdf/gazebo/transmission.xacro (robot description, xacro)
@@ -2,14 +2,12 @@
 <robot xmlns:xacro="http://ros.org/wiki/xacro" name="mobile_base">
     <xacro:macro name="wheel_transmission" params="joint_id">
-        <!-- Front left wheel -->
         <transmission name="${joint_id}_transmission">
-        <type>transmission_interface/SimpleTransmission</type>
-        <joint name="${joint_id}">
+          <type>transmission_interface/SimpleTransmission</type>
+          <joint name="${joint_id}">
             <hardwareInterface>hardware_interface/VelocityJointInterface</hardwareInterface>
-        </joint>
-        <actuator name="${joint_id}_motor">
-            <hardwareInterface>hardware_interface/VelocityJointInterface</hardwareInterface>
+          </joint>
+          <actuator name="${joint_id}_motor">
             <mechanicalReduction>1</mechanicalReduction>
-        </actuator>
+          </actuator>
         </transmission>
     </xacro:macro>

File: mobile_base_description/urdf/gazebo/wheel_physics.xacro (robot description, xacro)
@@ -16,6 +16,6 @@
         <xacro:wheel_physics joint_id="${frontLeftWheelId}"  friction_coeff="2.5"/>
         <xacro:wheel_physics joint_id="${frontRightWheelId}" friction_coeff="2.5"/>
-        <xacro:wheel_physics joint_id="${backLeftWheelId}"   friction_coeff="0.0"/>
-        <xacro:wheel_physics joint_id="${backRightWheelId}"  friction_coeff="0.0"/>
+        <xacro:wheel_physics joint_id="${backLeftWheelId}"   friction_coeff="2.5"/>
+        <xacro:wheel_physics joint_id="${backRightWheelId}"  friction_coeff="2.5"/>
     </xacro:macro>
 </robot>

File: mobile_base_description/urdf/mobile_base.urdf.xacro (robot description, xacro)
@@ -11,5 +11,5 @@
             <axis xyz="0 0 1" rpy="0 0 0" />
             <dynamics damping="1.0" friction="0.0"/>
-            <limit effort="1" velocity="1"/>
+            <limit effort="1000" velocity="1000"/>
             <joint_properties damping="0.2" friction="0.2"/>
         </joint>
@@ -50,5 +50,4 @@
                 <material name="green"/>
             </visual>
-            <inertial/>
         </link>
         <gazebo reference="base">

File: mobile_base_description/urdf/mobile_base_standalone.urdf.xacro (robot description, xacro)
@@ -2,5 +2,6 @@
 <robot xmlns:xacro="http://www.ros.org/wiki/xacro" name="mobile_base">
   <!-- Includes -->
-  <xacro:arg name="simulation" 			default="false"/>
+  <xacro:arg name="robot_name"          default="mobile_base"/>
+  <xacro:arg name="simulation" 			    default="false"/>
   <xacro:arg name="wheel_joint_type"  	default="fixed"/> <!-- continuous for gazebo -->
   <!-- Load the base -->
@@ -10,4 +11,5 @@
   <xacro:if value="$(arg simulation)">
     <xacro:include filename="$(find mobile_base_description)/urdf/gazebo/control.xacro"/>
+    <xacro:load_gazebo_ros_control ns="$(arg robot_name)"/>
   </xacro:if>
 </robot>
